File: ASM2001.sch (EAGLE design)
At the start: 18 parts, among them J1 3013, J2 DF12-32-DP, Q1 NTZD3152P, Q2 2N7002P, SW1 APTCLG, U1 ATMEGA328P, Y1 8MHz

Commit message: Updated to Rev6
Parts:
- added D3: MBR120, tinycircuits:AS-ITM-00111
- Q2: value 2N7002P -> 2N7002PT; device tinycircuits:AS-ITM-00007 -> tinycircuits:AS-ITM-00110; PARTNO AS-ITM-00007 -> (none)
Connections:
- new net N$2: D3.C, Q1.D2
- net +5V: now also D3.A; no longer Q1.D2
Other:
- note added: "6"
- note removed: "4"
- moved on the sheet: C1, R3

Commit message: Updated to Rev 8
Parts:
- removed Q1: NTZD3152P, tinycircuits:AS-ITM-00006
- added C5: 4.7uF, tinycircuits:AS-ITM-00242
- added D4: AMBER, tinycircuits:AS-ITM-00026
- added J3: 961102, tinycircuits:AS-ITM-00044
- added J4: SM02B-SRSS-TB(LF)(SN), tinycircuits:AS-ITM-00231
- added R6: 10K, tinycircuits:AS-ITM-00032
- added U2: MCP73831, tinycircuits:AS-ITM-00136
- C2: value 10uF -> .1uF; device tinycircuits:AS-ITM-00002 -> tinycircuits:AS-ITM-00008; PARTNO AS-ITM-00002 -> AS-ITM-00008; VALUE (none) -> 0.1uF
- C3: value .1uF -> 4.7uF; device tinycircuits:AS-ITM-00008 -> tinycircuits:AS-ITM-00242; PARTNO AS-ITM-00008 -> AS-ITM-00242; VALUE 0.1uF -> 4.7uF
- Q2: value 2N7002PT -> DMP2035U; device tinycircuits:AS-ITM-00110 -> tinycircuits:AS-ITM-00024
- R2: value 100k -> 1k; device tinycircuits:AS-ITM-00004 -> tinycircuits:AS-ITM-00003; PARTNO AS-ITM-00004 -> AS-ITM-00003; VALUE (none) -> 1.00K
- SW1: value APTCLG -> PCM12SMTR; device tinycircuits:AS-ITM-00010 -> tinycircuits:AS-ITM-00220; PARTNO AS-ITM-00010 -> (none)
- Y1: value 8MHz -> 8.00MHZ; device tinycircuits:AS-ITM-00027MU -> tinycircuits:AS-ITM-00027B
Connections:
- removed net N$8: Q1.G2, Q2.D, R2.1
- new net N$5: D4.C, R2.1
- new net N$6: R6.1, U2.PROG
- new net N$7: R2.2, U2.STAT
- net +5V: now also C5.1, D4.A, U2.VDD; no longer Q1.G1
- net AREF: no longer C3.1
- net GND: now also C5.2, J3.2, J4.2, R6.2, SW1.TAB, U2.VSS; no longer Q2.S, SW1.2, SW1.4, SW1.5
- net N$2: now also Q2.S, SW1.1; no longer Q1.D2
- net RESET: no longer SW1.1, SW1.3
- net VBATT: now also C3.1, J3.1, J4.1, Q2.D, U2.VBAT; no longer C2.1, J1.1, Q1.D1
- net VCC: now also C2.1, SW1.2; no longer Q1.S1, Q1.S2, R2.2
Other:
- note added: "8"
- note added: "Battery Connections"
- note added: "Lithium Battery Charger"
- note removed: "6"
- moved on the sheet: C1, C2, C3, C4, D1, D2, D3, J1, J2, R1, R2, R3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

Commit message: Update to Rev 9
Parts:
- C5: value 4.7uF -> 10uF; device tinycircuits:AS-ITM-00242 -> tinycircuits:AS-ITM-00002; PARTNO AS-ITM-00242 -> AS-ITM-00002; VALUE 4.7uF -> 10uF
Other:
- note added: "9"
- note removed: "8"
Changed lines of the file:
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@@
 <part name="VBATT4" library="tinycircuits" deviceset="VBATT" device="" value="VBATT"/>
 <part name="GND13" library="tinycircuits" deviceset="GND" device=""/>
-<part name="C5" library="tinycircuits" deviceset="AS-ITM-00242" device="" value="4.7uF">
-<attribute name="PARTNO" value="AS-ITM-00242"/>
-<attribute name="VALUE" value="4.7uF"/>
+<part name="C5" library="tinycircuits" deviceset="AS-ITM-00002" device="" value="10uF">
+<attribute name="PARTNO" value="AS-ITM-00002"/>
+<attribute name="VALUE" value="10uF"/>
 </part>
 <part name="GND14" library="tinycircuits" deviceset="GND" device=""/>
@@
 <text x="340.868" y="17.272" size="3.556" layer="94" font="vector">TinyDuino - 20mm</text>
 <text x="327.152" y="6.35" size="3.556" layer="94" font="vector">AS-SCH-ASM2001</text>
-<text x="416.56" y="6.858" size="3.556" layer="94" font="vector">8</text>
+<text x="416.56" y="6.858" size="3.556" layer="94" font="vector">9</text>
 <text x="45.72" y="35.56" size="3.048" layer="91">Released under the Creative Commons Attribution Share-Alike 3.0 License</text>
 <text x="45.72" y="30.48" size="3.048" layer="91">http://creativecommons.org/licenses/by-sa/3.0</text>
